File: DP100.kicad_pcb (KiCad board)
At the start: 2 copper layers, 36 x 46 mm, 60 parts, among them J1 SMA CONNECTOR, J2 Conn_01x06, J3 Conn_02x06_Odd_Even, Q1 2N7002, U1 NCP1117-3.3_SOT223, U2 Si5351A-B-GT, U3 AD9215BRUZ, Y1 25MHZ

Commit message: Se agregan correcciones realizadas por Francisco Timez el dia 10-4 -Fiduciarios -Serigrafias faltantes -Otro agujero de sujecion
Parts:
- added FID1: Fiducial, Fiducial:Fiducial_0.5mm_Mask1mm, F.Cu at (142.0, 120.5)
- added H1: MountingHole, MountingHole:MountingHole_3mm, F.Cu at (113.0, 150.0)
- added H2: MountingHole, MountingHole:MountingHole_3mm, F.Cu at (113.0, 112.0)
Routing:
- net (no net): vias 1 -> 0
Other:
- board text added: "5V"
- board text added: "CLK"
- board text added: "D0"
- board text added: "D1"
- board text added: "D2"
- board text added: "D3"
- board text added: "D4"
- board text added: "D5"
- board text added: "D6"
- board text added: "D7"
- board text added: "D8"
- board text added: "DISEÑADO EN ARGENTINA"
- board text added: "GND"
- board text added: "OR"
- board text added: "PWDWN"
- board text added: "SCL"
- board text added: "SDA"
- board text added: "SP"
- board text added: "V1.0"
Changed lines of the file:
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@@
   (general
     (thickness 1.6)
-    (drawings 23)
-    (tracks 380)
+    (drawings 43)
+    (tracks 379)
     (zones 0)
-    (modules 60)
+    (modules 63)
     (nets 51)
   )
   (page A4)
   (layers
-    (0 F.Cu signal hide)
-    (31 B.Cu signal hide)
+    (0 F.Cu signal)
+    (31 B.Cu signal)
     (32 B.Adhes user)
     (33 F.Adhes user)
@@
     (uvia_drill 0.4)
   )
+  (module Fiducial:Fiducial_0.5mm_Mask1mm (layer F.Cu)
+    (at 142 120.5)
+    (descr "Circular Fiducial, 0.5mm bare copper, 1mm soldermask opening (Level C)")
+    (tags fiducial)
+    (attr smd)
+    (fp_text reference FID1 (at 0 -1.5) (layer F.SilkS)
+      (effects (font (size 1 1) (thickness 0.15)))
+    )
+    (fp_text value Fiducial (at 0 1.5) (layer F.Fab)
+      (effects (font (size 1 1) (thickness 0.15)))
+    )
+    (fp_circle (center 0 0) (end 0.75 0) (layer F.CrtYd) (width 0.05))
+    (fp_text user %R (at 0 0) (layer F.Fab)
+      (effects (font (size 0.2 0.2) (thickness 0.04)))
+    )
+    (fp_circle (center 0 0) (end 0.5 0) (layer F.Fab) (width 0.1))
+    (pad "" smd circle (at 0 0) (size 0.5 0.5) (layers F.Cu F.Mask)
+      (solder_mask_margin 0.25) (clearance 0.25))
+  )
+  (module MountingHole:MountingHole_3mm (layer F.Cu)
+    (at 113 112)
+    (descr "Mounting Hole 3mm, no annular")
+    (tags "mounting hole 3mm no annular")
+    (attr virtual)
+    (fp_text reference H2 (at 4.6 0) (layer F.SilkS)
+      (effects (font (size 1 1) (thickness 0.15)))
+    )
+    (fp_text value MountingHole (at 0 4) (layer F.Fab)
+      (effects (font (size 1 1) (thickness 0.15)))
+    )
+    (fp_circle (center 0 0) (end 3.25 0) (layer F.CrtYd) (width 0.05))
+    (fp_circle (center 0 0) (end 3 0) (layer Cmts.User) (width 0.15))
+    (fp_text user %R (at 0.3 0) (layer F.Fab)
+      (effects (font (size 1 1) (thickness 0.15)))
+    )
+    (pad 1 np_thru_hole circle (at 0 0) (size 3 3) (drill 3) (layers *.Cu *.Mask))
+  )
+  (module MountingHole:MountingHole_3mm (layer F.Cu)
+    (at 113 150)
+    (descr "Mounting Hole 3mm, no annular")
+    (tags "mounting hole 3mm no annular")
+    (attr virtual)
+    (fp_text reference H1 (at 4.6 0) (layer F.SilkS)
+      (effects (font (size 1 1) (thickness 0.15)))
+    )
+    (fp_text value MountingHole (at 0 4) (layer F.Fab)
+      (effects (font (size 1 1) (thickness 0.15)))
+    )
+    (fp_circle (center 0 0) (end 3.25 0) (layer F.CrtYd) (width 0.05))
+    (fp_circle (center 0 0) (end 3 0) (layer Cmts.User) (width 0.15))
+    (fp_text user %R (at 0.3 0) (layer F.Fab)
+      (effects (font (size 1 1) (thickness 0.15)))
+    )
+    (pad 1 np_thru_hole circle (at 0 0) (size 3 3) (drill 3) (layers *.Cu *.Mask))
+  )
   (module Resistor_SMD:R_0603_1608Metric_Pad1.05x0.95mm_HandSolder (layer F.Cu)
     (at 124.4 118.495 270)
@@
     (attr smd)
     (fp_text reference L4 (at -0.025 0 90) (layer F.SilkS)
-      (effects (font (size 1 1) (thickness 0.15)))
+      (effects (font (size 0.6 0.6) (thickness 0.15)))
     )
     (fp_text value 455nH (at 0 1.65) (layer F.Fab)
@@
     (attr smd)
     (fp_text reference L3 (at 0 0 90) (layer F.SilkS)
-      (effects (font (size 1 1) (thickness 0.15)))
+      (effects (font (size 0.6 0.6) (thickness 0.15)))
     )
     (fp_text value 455nH (at 0 1.65) (layer F.Fab)
@@
     )
   )
+  (gr_text V1.0 (at 130.8 113) (layer B.SilkS)
+    (effects (font (size 1 1) (thickness 0.15)) (justify mirror))
+  )
+  (gr_text OR (at 137 142.4 90) (layer B.SilkS)
+    (effects (font (size 1 1) (thickness 0.15)) (justify mirror))
+  )
+  (gr_text D8 (at 134.4 142.4 90) (layer B.SilkS)
+    (effects (font (size 1 1) (thickness 0.15)) (justify mirror))
+  )
+  (gr_text D6 (at 132 142.4 90) (layer B.SilkS)
+    (effects (font (size 1 1) (thickness 0.15)) (justify mirror))
+  )
+  (gr_text D4 (at 129.4 142.4 90) (layer B.SilkS)
+    (effects (font (size 1 1) (thickness 0.15)) (justify mirror))
+  )
+  (gr_text D2 (at 127 142.4 90) (layer B.SilkS)
+    (effects (font (size 1 1) (thickness 0.15)) (justify mirror))
+  )
+  (gr_text D0 (at 124.4 142.4 90) (layer B.SilkS)
+    (effects (font (size 1 1) (thickness 0.15)) (justify mirror))
+  )
+  (gr_text SP (at 137 145 90) (layer B.SilkS)
+    (effects (font (size 1 1) (thickness 0.15)) (justify mirror))
+  )
+  (gr_text D8 (at 134.4 145 90) (layer B.SilkS)
+    (effects (font (size 1 1) (thickness 0.15)) (justify mirror))
+  )
+  (gr_text D7 (at 132 145 90) (layer B.SilkS)
+    (effects (font (size 1 1) (thickness 0.15)) (justify mirror))
+  )
+  (gr_text D5 (at 129.4 145 90) (layer B.SilkS)
+    (effects (font (size 1 1) (thickness 0.15)) (justify mirror))
+  )
+  (gr_text D3 (at 127 145 90) (layer B.SilkS)
+    (effects (font (size 1 1) (thickness 0.15)) (justify mirror))
+  )
+  (gr_text D1 (at 124.4 145 90) (layer B.SilkS)
+    (effects (font (size 1 1) (thickness 0.15)) (justify mirror))
+  )
+  (gr_text SDA (at 115 134) (layer B.SilkS)
+    (effects (font (size 1 1) (thickness 0.15)) (justify mirror))
+  )
+  (gr_text SCL (at 115 131.2) (layer B.SilkS)
+    (effects (font (size 1 1) (thickness 0.15)) (justify mirror))
+  )
+  (gr_text CLK (at 115 128.8) (layer B.SilkS)
+    (effects (font (size 1 1) (thickness 0.15)) (justify mirror))
+  )
+  (gr_text PWDWN (at 116 126.2) (layer B.SilkS)
+    (effects (font (size 1 1) (thickness 0.15)) (justify mirror))
+  )
+  (gr_text 5V (at 114.5 123.6) (layer B.SilkS)
+    (effects (font (size 1 1) (thickness 0.15)) (justify mirror))
+  )
+  (gr_text GND (at 115 121.2) (layer B.SilkS)
+    (effects (font (size 1 1) (thickness 0.15)) (justify mirror))
+  )
+  (gr_text HSADC100 (at 126.8 110.6) (layer B.SilkS)
+    (effects (font (size 1.5 1.5) (thickness 0.15)) (justify mirror))
+  )
+  (gr_text "DISEÑADO EN ARGENTINA" (at 123.2 117) (layer B.SilkS)
+    (effects (font (size 1 1) (thickness 0.15)) (justify mirror))
+  )
   (dimension 46 (width 0.15) (layer Dwgs.User)
     (gr_text "46,000 mm" (at 102.7 131 90) (layer Dwgs.User)
@@
     (arrow2a (pts (xy 109 103) (xy 110.126504 103.586421)))
     (arrow2b (pts (xy 109 103) (xy 110.126504 102.413579)))
-  )
-  (gr_text HSADC100 (at 116.2 148.6) (layer F.SilkS)
-    (effects (font (size 1.5 1.5) (thickness 0.15)))
   )
   (gr_line (start 125 135.6) (end 125.8 134.8) (layer F.SilkS) (width 0.12))
@@
   (gr_line (start 145 154) (end 145 108) (layer Edge.Cuts) (width 0.05))
   (gr_line (start 109 154) (end 145 154) (layer Edge.Cuts) (width 0.05))
-  (via (at 114 112) (size 4.1) (drill 4) (layers F.Cu B.Cu) (net 0))
   (via (at 120.8 123.6) (size 0.8) (drill 0.4) (layers F.Cu B.Cu) (net 1))
   (segment (start 122 125.85) (end 120.7 124.55) (width 0.5) (layer F.Cu) (net 1))
@@
   (via (at 117 150.4) (size 0.8) (drill 0.4) (layers F.Cu B.Cu) (net 2))
   (via (at 118.2 150.4) (size 0.8) (drill 0.4) (layers F.Cu B.Cu) (net 2))
-  (via (at 115.8 150.4) (size 0.8) (drill 0.4) (layers F.Cu B.Cu) (net 2))
-  (via (at 114.6 150.4) (size 0.8) (drill 0.4) (layers F.Cu B.Cu) (net 2))
+  (via (at 120.6 150.4) (size 0.8) (drill 0.4) (layers F.Cu B.Cu) (net 2))
+  (via (at 119.4 150.4) (size 0.8) (drill 0.4) (layers F.Cu B.Cu) (net 2))
   (via (at 111.6 117.2) (size 0.8) (drill 0.4) (layers F.Cu B.Cu) (net 2))
   (via (at 113 117.2) (size 0.8) (drill 0.4) (layers F.Cu B.Cu) (net 2))
@@
   (via (at 129 130.8) (size 0.8) (drill 0.4) (layers F.Cu B.Cu) (net 7))
   (segment (start 131.6 134) (end 132.075 134) (width 0.4) (layer F.Cu) (net 7))
-  (via (at 133.675 132) (size 0.8) (drill 0.4) (layers F.Cu B.Cu) (net 7) (status 1000000))
+  (via (at 133.675 132) (size 0.8) (drill 0.4) (layers F.Cu B.Cu) (net 7))
   (segment (start 133.675 132.725) (end 133.675 132) (width 0.4) (layer F.Cu) (net 7))
   (segment (start 132.4 134) (end 133.675 132.725) (width 0.4) (layer F.Cu) (net 7))

Commit message: Correcciones en base a devolucion de Diego Brengi del dia 12-4-2021 -Se expanden las zonas compactas -Se agrega directorio con informacion extra -Se agregan lineas para evitar que los labels toquen directamente el componente -Se agrega bus para unir los pines Dn -Se agrega referencia  a la licencia -Se remueven las etiquetas filterIn
Connections:
- net /filterIn+ renamed Net-(C2-Pad2)
- net /filterIn- renamed Net-(C3-Pad2)
